File: demo_board/DDL_demo_board.sch (EAGLE design)
At the start: 36 parts, among them IC1 74LS14N

Commit message: Updated demo board for new inductors * added gerbers to repository * added zip file script
Parts:
- removed U$31: Z0_LOGO200MIL_NO_Z, z0:Z0_LOGO200MIL_NO_Z
- C1: value (none) -> 1n
- C10, C11, C6, C7, C8, C9: value (none) -> 10n
- C2, C3: value (none) -> 100n
- C4: value (none) -> 10u
- L1, L2: value (none) -> 47u; device z0:L-US0204/5 -> z0:L-US0207/10
- LED1, LED2: value (none) -> WP7113SRD/E
- R1, R2, R3, R4: value (none) -> 39
- R5, R6, R7: value (none) -> 220
- R8: value (none) -> 1k
